File: mm_motor_control.kicad_sch (KiCad schematic)
At the start: 0 parts

Commit message: fin tp2
Parts:
- added C10: 22 nF, symbol Device:C
- added C11: 2.2 uF / 16V, symbol Device:C
- added C12: 22 uF / 16 V, symbol Device:C
- added C7: 10 uF, symbol Device:C
- added C8: 10 nF / 6.3 V, symbol Device:C
- added C9: 1 nF / 6.3 V, symbol Device:C
- added R1, R2: 10 KOhms, symbol Device:R
- added R3: 18 KOhms, symbol Device:R
- added R4: 18 KHoms, symbol Device:R
- added R5: 1 KOhms, symbol Device:R
- added R6: 47 KHoms, symbol Device:R
- added R7, R8: 330 mOhms, symbol Device:R
- added U2: STSPIN240, Package_DFN_QFN:VQFN-16-1EP_3x3mm_P0.5mm_EP1.8x1.8mm, symbol Driver_Motor:STSPIN240
Connections:
- net EN: now also R3.2
- net OUT_A1: now also U2.3 (OUTA1)
- net OUT_A2: now also U2.5 (OUTA2)
- net OUT_B1: now also U2.10 (OUTB1)
- net OUT_B2: now also U2.8 (OUTB2)
- net PHASE_A: now also U2.1 (PHA)
- net PHASE_B: now also U2.15 (PHB)
- net PWM_A: now also U2.2 (PWMA)
- net PWM_B: now also U2.16 (PWMB)
- net STBY/RESET: now also C9.1, R4.2, U2.14 (STBY/RESET)
- new net: R5.1, R6.1, U2.12 (TOFF)
- new net: C10.1, R5.2
- new net: R8.1, U2.9 (SENSEB)
- new net: R7.1, U2.4 (SENSEA)
- new net +3.3V: R4.1
- new net +BATT: C11.1, C12.1, C7.1, R1.1, U2.6 (VS)
- new net EN / FLT: R1.2, R2.1, U2.13 (EN/FLT)
- new net GND: C10.2, C11.2, C12.2, C7.2, C8.2, C9.2, R2.2, R6.2, R7.2, R8.2, U2.17 (EPAD), U2.7 (GND)
- new net REF: C8.1, R3.1, U2.11 (REF)
