File: mm_power.kicad_sch (KiCad schematic)
At the start: 1 part, among them J5 Conn_01x02

Commit message: fin tp2
Parts:
- added C7, C8: 22 uF, symbol Device:C
- added D1: LED, symbol Device:LED
- added R0: 180 Ohms, symbol Device:R
- added U3: LP5907MFX-1.2, Package_TO_SOT_SMD:SOT-23-5, symbol Regulator_Linear:LP5907MFX-1.2
Connections:
- net +BATT: now also C7.1, U3.1 (IN), U3.3 (EN)
- net GND: now also C7.2, C8.2, R0.2, U3.2 (GND)
- new net: D1.1 (K), R0.1
- new net +3.3V: C8.1, D1.2 (A), U3.5 (OUT)

Commit message: TP
Parts:
- C1: renamed from C7; value 22 uF -> 2.2 uF; footprint (none) -> Capacitor_SMD:C_0603_1608Metric
- C2: renamed from C8; value 22 uF -> 2.2 uF; footprint (none) -> Capacitor_SMD:C_0603_1608Metric
- D1: footprint (none) -> LED_SMD:LED_0603_1608Metric
- R1: renamed from R0; value 180 Ohms -> 330; footprint (none) -> Resistor_SMD:R_0603_1608Metric
- renumbered J5 to J1, U3 to U1
