File: tp3.kicad_pcb (KiCad board)
At the start: 2 copper layers, 90 x 85 mm, 52 parts, among them J1 Conn_01x02, J2 Conn_ARM_JTAG_SWD_10, J3 Conn_01x06, J4 Conn_01x06, J5 Conn_01x04, M1 N20_encoder, M2 N20_encoder, U1 LP5907MFX-1.2, U2 STM32F030C8Tx, U3 STSPIN240, U4 HC-SR04

Commit message: tp5
Parts:
- removed the R7 at (137.3, 90.1)
- added BOOT2: RESET, TestPoint:TestPoint_Pad_D1.5mm, F.Cu at (1.27, 1.27)
- moved R13 23.2 mm to (161.9, 83.3)
- moved R15 23.1 mm to (165.3, 98.7)
- moved R18 23.0 mm to (169.5, 100.0)
- moved R16 22.7 mm to (160.2, 92.3)
- moved C10 22.6 mm to (166.6, 84.4), turned to -90 degrees
- moved R17 21.5 mm to (165.8, 100.9), turned to 0 degrees
- moved R14 20.5 mm to (161.8, 85.3), turned to 0 degrees
- moved C11 18.4 mm to (162.7, 96.1)
- moved R11 18.4 mm to (158.8, 88.7), turned to 0 degrees
- moved R12 16.3 mm to (160.3, 90.5), turned to 180 degrees
- moved R7 11.7 mm to (145.6, 88.0), turned to 180 degrees
- moved J4 11.2 mm to (136.9, 103.8)
- moved C12 10.6 mm to (171.9, 99.9)
- moved J3 10.6 mm to (161.8, 103.8)
- moved R5 8.68 mm to (149.0, 73.2), turned to -90 degrees
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Connections:
- J5 pad 4: /external_uart/UART1_RX -> /external_uart/EXT_UART_RX
- R21 pad 1: /external_uart/UART1_TX -> /external_uart/EXT_UART_TX
- R22 pad 1: /mcu/TIM8_CH2 -> Net-(U4-ECHO)
- R22 pad 2: Net-(U4-ECHO) -> /mcu/TIM8_CH2
- R4 pad 1: /mcu/UART1_TX -> /external_uart/EXT_UART_RX
- U2 pad 43: /mcu/UART1_RX -> /external_uart/EXT_UART_TX
- U4 pad 4: +3V3 -> +BATT
Routing:
- net +BATT: track 13.3 -> 113.3 mm
- net GND: track 2.77 -> 98.0 mm, vias 0 -> 10
- net /mcu/~{RESET}: track 0.00 -> 34.4 mm, vias 0 -> 2
- net /mcu/TIM2_CH2: track 0.00 -> 29.0 mm, vias 0 -> 2
- net /mcu/TIM2_CH1: track 0.00 -> 27.0 mm
- net /mcu/TIM3_CH2: track 6.61 -> 33.4 mm
- net /mcu/TIM3_CH1: track 8.04 -> 31.6 mm
- net /mcu/SWO: track 0.00 -> 21.5 mm
- net /mcu/SWDCLK: track 0.00 -> 19.0 mm
- net Net-(U3-TOFF): track 0.00 -> 18.7 mm
- net Net-(J3-Pin_4): track 21.3 -> 3.07 mm
- net Net-(J3-Pin_3): track 20.7 -> 3.16 mm
- net /mcu/SWDIO: track 0.00 -> 17.5 mm
- net Net-(U2-PA4): track 0.00 -> 10.5 mm
- net Net-(U2-PA2): track 0.00 -> 9.20 mm
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